File: H7_FOC_Project/H7_Board/H7_Board.kicad_pcb (KiCad board)
At the start: 2 copper layers, 63 parts, among them J1 Conn_ARM_JTAG_SWD_10, J10 PWR_CON, J2 PWM_CON, J3 ADC_CON, J4 Add_ADC_CON, J5 SETTING_CON, J6 USER_DEBUG_CON, J7 SPI5_CON, J8 ABZ_ENC, J9 UI_CON, SW1 RST_SW, U1 LD1117S33TR_SOT223, U2 STM32H743ZITx, Y1 8M, Y2 32K

Commit message: [fix] schematic
Parts:
- removed J10: PWR_CON, Connector_PinSocket_1.27mm:PinSocket_2x05_P1.27mm_Vertical_SMD
- removed J9: UI_CON, Connector_PinSocket_1.27mm:PinSocket_2x05_P1.27mm_Vertical_SMD
- removed JP3: SolderBridge, Jumper:SolderJumper-2_P1.3mm_Open_TrianglePad1.0x1.5mm
- added D12: ESDA6V1-5SC6, Package_TO_SOT_SMD:SOT-23-6, F.Cu at (79.8, 67.6)
- added D13: ESDA6V1-5SC6, Package_TO_SOT_SMD:SOT-23-6, F.Cu at (131.6, 31.6)
- added D14: ESDA6V1-5SC6, Package_TO_SOT_SMD:SOT-23-6, F.Cu at (103.4, 58.5)
- C24, C25: value 5p -> 18p
- C26, C27: value 5p -> 12.5p
- D1: value D_ESD -> LED; footprint Diode_SMD:D_MELF -> LED_SMD:LED_0603_1608Metric
- D10, D11, D9: value LED -> ESDA6V1-5SC6; footprint LED_SMD:LED_0603_1608Metric -> Package_TO_SOT_SMD:SOT-23-6
- D2, D3: value ESDA6V1-5SC6 -> LED; footprint Package_TO_SOT_SMD:SOT-23-6 -> LED_SMD:LED_0603_1608Metric
- D4: value ESDA6V1-5SC6 -> D_ESD; footprint Package_TO_SOT_SMD:SOT-23-6 -> Diode_SMD:D_MELF
- D5, D6, D7: value ESDA6V1-5SC6 -> SBD; footprint Package_TO_SOT_SMD:SOT-23-6 -> Diode_SMD:D_MELF
- J4: value Add_ADC_CON -> SETTING_CON
- J5: value SETTING_CON -> USER_DEBUG_CON
- J6: value USER_DEBUG_CON -> ENC_CON
- J7: value SPI5_CON -> PWR_CON
- J8: value ABZ_ENC -> UI_CON
- Y1: value 8M -> 8M RH100-8.000-20-3050-EXT-TR; footprint Crystal:Crystal_SMD_0603-4Pin_6.0x3.5mm -> Crystal:Crystal_SMD_3225-4Pin_3.2x2.5mm
- Y2: value 32K -> 32k FC-135 32.7680KA-A0; footprint Crystal:Crystal_SMD_0603-4Pin_6.0x3.5mm -> Crystal:Crystal_SMD_3215-2Pin_3.2x1.5mm
- moved J1 137.1 mm to (164.5, 49.9), turned to 180 degrees
- moved U2 112.1 mm to (146.2, 74.5)
- moved C9 75.0 mm to (179.0, 63.9)
- moved C16 70.5 mm to (170.9, 61.5)
- moved R6 69.5 mm to (170.1, 69.0)
- moved C4 62.1 mm to (167.1, 75.1)
- moved C23 61.3 mm to (166.1, 70.1)
- moved C27 59.1 mm to (174.9, 61.9)
- moved C26 58.8 mm to (149.1, 51.2)
- moved C3 58.1 mm to (170.9, 66.5)
- moved C13 55.8 mm to (179.0, 61.3)
- moved C6 55.6 mm to (174.9, 66.9)
- moved C20 55.5 mm to (166.9, 66.5)
- moved JP1 54.2 mm to (65.9, 58.4)
- moved D11 53.2 mm to (122.1, 29.7)
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Connections:
- C21 pad 1: /NRST -> /NJTRST
- D1 pad 1: /NRST -> Net-(D1-Pad1)
- D1 pad 2: GND -> /LED1
- D10 pad 1: Net-(D10-Pad1) -> /SPI5_NSS
- D10 pad 2: /LED2 -> GND
- D11 pad 1: Net-(D11-Pad1) -> /Start_Stop
- D11 pad 2: /LED3 -> GND
- D2 pad 1: /PG_TRG -> Net-(D2-Pad1)
- D2 pad 2: GND -> /LED2
- D3 pad 1: /SPI4_NSS -> Net-(D3-Pad1)
- D3 pad 2: GND -> /LED3
- D4 pad 1: /SPI5_NSS -> /NJTRST
- D5 pad 1: /Start_Stop -> Net-(D5-Pad1)
- D5 pad 2: GND -> /3V3_VDD
- D6 pad 1: /NJTRST -> Net-(D6-Pad1)
- D6 pad 2: GND -> /3V3_VDD
- D7 pad 1: /UART_TX -> Net-(D7-Pad1)
- D7 pad 2: GND -> /5V_IN
- D8 pad 1: /UI_PIN_4 -> /PG_TRG
- D8 pad 3: /UI_PIN_5 -> /Fault_TRG
- D8 pad 4: /UI_PIN_6 -> /OC_TRG
- D8 pad 5: /UI_PIN_7 -> /ABZ_ENC_A
- D8 pad 6: /UI_PIN_8 -> /ABZ_ENC_B
- D9 pad 1: Net-(D9-Pad1) -> /SPI4_NSS
- D9 pad 2: /LED1 -> GND
- J1 pad 7: Net-(J1-Pad7) -> (no net)
- J3 pad 2: GND -> /Add_ADC3
- J3 pad 3: GND -> /ADC_V
- J3 pad 4: GND -> /Add_ADC4
- J3 pad 5: /ADC_V -> /ADC_W
- J3 pad 7: GND -> /Add_ADC1
- J3 pad 9: /ADC_W -> /Add_ADC2
- J4 pad 1: /Add_ADC1 -> /Gate_Enable
- J4 pad 2: GND -> /OC_TRG
- J4 pad 3: GND -> /PWM_MODE
- J4 pad 4: /Add_ADC4 -> /Fault_TRG
- J4 pad 5: /Add_ADC2 -> /OC_MODE
- J4 pad 6: GND -> /PG_TRG
- J4 pad 9: /Add_ADC3 -> /CurrentLimit
- J5 pad 1: /Gate_Enable -> /SPI4_NSS
- J5 pad 2: /OC_TRG -> /UART_TX
- J5 pad 3: /PWM_MODE -> /SPI4_SCK
- J5 pad 4: /Fault_TRG -> /UART_RX
- J5 pad 5: /OC_MODE -> /SPI4_MISO
- J5 pad 6: /PG_TRG -> /CAN_TX
- J5 pad 7: GND -> /SPI4_MOSI
- J5 pad 8: GND -> /CAN_RX
- J5 pad 9: /CurrentLimit -> Net-(D5-Pad1)
- J6 pad 1: /SPI4_NSS -> /SPI5_NSS
- J6 pad 10: /CAN_RX -> GND
- J6 pad 2: /UART_TX -> /ABZ_ENC_B
- J6 pad 3: /SPI4_SCK -> /SPI5_SCK
- J6 pad 4: /UART_RX -> /ABZ_ENC_A
- J6 pad 5: /SPI4_MISO -> /SPI5_MISO
- J6 pad 6: GND -> /ABZ_ENC_GPIO
- J6 pad 7: /SPI4_MOSI -> /SPI5_MOSI
- J6 pad 8: /CAN_TX -> Net-(D7-Pad1)
- J6 pad 9: GND -> Net-(D6-Pad1)
- J7 pad 1: /SPI5_NSS -> /5V_IN
- J7 pad 10: Net-(J7-Pad10) -> GND
- J7 pad 2: Net-(J7-Pad2) -> GND
- J7 pad 3: /SPI5_SCK -> /5V_IN
- J7 pad 4: Net-(J7-Pad4) -> GND
- J7 pad 5: /SPI5_MISO -> /5V_IN
- J7 pad 6: Net-(J7-Pad6) -> GND
- J7 pad 7: /SPI5_MOSI -> /5V_IN
- J7 pad 8: Net-(J7-Pad8) -> GND
- J7 pad 9: Net-(J7-Pad9) -> /5V_IN
- J8 pad 1: /ABZ_ENC_A -> /Start_Stop
- J8 pad 10: Net-(J8-Pad10) -> /UI_PIN_8
- J8 pad 2: Net-(J8-Pad2) -> /UI_PIN_4
- J8 pad 3: /ABZ_ENC_B -> /Stop
- J8 pad 4: Net-(J8-Pad4) -> /UI_PIN_5
- J8 pad 5: Net-(J8-Pad5) -> /UI_PIN_1
- J8 pad 6: Net-(J8-Pad6) -> /UI_PIN_6
- J8 pad 7: Net-(J8-Pad7) -> /UI_PIN_2
- J8 pad 8: Net-(J8-Pad8) -> /UI_PIN_7
- J8 pad 9: Net-(J8-Pad9) -> /UI_PIN_3
- R3 pad 1: GND -> Net-(D1-Pad1)
- R3 pad 2: /BOOT0 -> GND
- R4 pad 1: Net-(R4-Pad1) -> Net-(D2-Pad1)
- R4 pad 2: /3V3_VDD -> GND
- R5 pad 1: Net-(D9-Pad1) -> Net-(D3-Pad1)
- R6 pad 1: Net-(D10-Pad1) -> GND
- R6 pad 2: GND -> /BOOT0
- R7 pad 1: Net-(D11-Pad1) -> Net-(R7-Pad1)
- R7 pad 2: GND -> /3V3_VDD
- SW1 pad 2: /NRST -> /NJTRST
- U2 pad 100: Net-(U2-Pad100) -> (no net)
- U2 pad 101: Net-(U2-Pad101) -> (no net)
- U2 pad 102: Net-(U2-Pad102) -> (no net)
- U2 pad 103: Net-(U2-Pad103) -> (no net)
- U2 pad 104: Net-(U2-Pad104) -> (no net)
- U2 pad 111: Net-(U2-Pad111) -> (no net)
- U2 pad 112: Net-(U2-Pad112) -> (no net)
- U2 pad 124: Net-(U2-Pad124) -> (no net)
- U2 pad 125: Net-(U2-Pad125) -> (no net)
- U2 pad 126: Net-(U2-Pad126) -> (no net)
- U2 pad 127: Net-(U2-Pad127) -> (no net)
- U2 pad 128: Net-(U2-Pad128) -> (no net)
- U2 pad 129: Net-(U2-Pad129) -> (no net)
- U2 pad 13: Net-(U2-Pad13) -> (no net)
- U2 pad 132: Net-(U2-Pad132) -> (no net)
- U2 pad 135: Net-(U2-Pad135) -> (no net)
- U2 pad 136: Net-(U2-Pad136) -> (no net)
- U2 pad 139: Net-(U2-Pad139) -> (no net)
- U2 pad 14: Net-(U2-Pad14) -> (no net)
- U2 pad 140: Net-(U2-Pad140) -> (no net)
- U2 pad 141: Net-(U2-Pad141) -> (no net)
- U2 pad 143: Net-(R4-Pad1) -> Net-(R7-Pad1)
- U2 pad 15: Net-(U2-Pad15) -> (no net)
- U2 pad 2: Net-(U2-Pad2) -> (no net)
- U2 pad 25: /NRST -> /NJTRST
- U2 pad 26: Net-(U2-Pad26) -> (no net)
- U2 pad 27: Net-(U2-Pad27) -> (no net)
- U2 pad 33: Net-(JP3-Pad2) -> /VDDA
- U2 pad 34: Net-(U2-Pad34) -> (no net)
- U2 pad 35: Net-(U2-Pad35) -> (no net)
- U2 pad 36: Net-(U2-Pad36) -> (no net)
- U2 pad 37: Net-(U2-Pad37) -> (no net)
- U2 pad 41: Net-(U2-Pad41) -> (no net)
- U2 pad 43: Net-(U2-Pad43) -> (no net)
- U2 pad 44: Net-(U2-Pad44) -> (no net)
- U2 pad 45: Net-(U2-Pad45) -> (no net)
- U2 pad 48: Net-(U2-Pad48) -> (no net)
- U2 pad 49: Net-(U2-Pad49) -> (no net)
- U2 pad 50: Net-(U2-Pad50) -> (no net)
- U2 pad 55: Net-(U2-Pad55) -> (no net)
- U2 pad 56: Net-(U2-Pad56) -> (no net)
- U2 pad 57: Net-(U2-Pad57) -> (no net)
- U2 pad 58: Net-(U2-Pad58) -> (no net)
- U2 pad 73: Net-(U2-Pad73) -> (no net)
- U2 pad 74: Net-(U2-Pad74) -> (no net)
- U2 pad 76: Net-(U2-Pad76) -> (no net)
- U2 pad 79: Net-(U2-Pad79) -> (no net)
- U2 pad 80: Net-(U2-Pad80) -> (no net)
- U2 pad 85: Net-(U2-Pad85) -> /ABZ_ENC_GPIO
- U2 pad 86: Net-(U2-Pad86) -> (no net)
- U2 pad 87: Net-(U2-Pad87) -> (no net)
- U2 pad 88: Net-(U2-Pad88) -> (no net)
- U2 pad 89: Net-(U2-Pad89) -> (no net)
- U2 pad 90: Net-(U2-Pad90) -> (no net)
- U2 pad 91: Net-(U2-Pad91) -> (no net)
- U2 pad 92: Net-(U2-Pad92) -> (no net)
- U2 pad 93: Net-(U2-Pad93) -> (no net)
- U2 pad 96: Net-(U2-Pad96) -> (no net)
- U2 pad 97: Net-(U2-Pad97) -> (no net)
- U2 pad 98: Net-(U2-Pad98) -> (no net)
- U2 pad 99: Net-(U2-Pad99) -> (no net)
- Y1 pad 3: GND -> Net-(C25-Pad1)
- Y1 pad 4: Net-(C25-Pad1) -> GND
- Y2 pad 1: Net-(C27-Pad1) -> Net-(C26-Pad1)
- Y2 pad 2: GND -> Net-(C27-Pad1)

Commit message: [modify] CAD
Parts:
- removed the C10 at (104.5, 66.2)
- removed the C12 at (171.1, 71.5)
- removed the C15 at (166.9, 61.5)
- removed the C2 at (167.1, 72.6)
- removed the C20 at (166.9, 66.5)
- removed the C24 at (113.9, 54.3)
- removed the C25 at (120.7, 81.2)
- removed the C27 at (174.9, 61.9)
- removed the C3 at (170.9, 66.5)
- removed the C4 at (167.1, 75.1)
- removed the C5 at (153.1, 53.7)
- removed the C6 at (174.9, 66.9)
- removed the C7 at (121.9, 52.7)
- removed the C8 at (61.5, 58.1)
- removed the C9 at (179.0, 63.9)
- removed the Y1 at (130.4, 77.0)
- added C1: 0.1u, Capacitor_SMD:C_0402_1005Metric, F.Cu at (-113.1, 44.2)
- added C1: 0.1u, Capacitor_SMD:C_0402_1005Metric, F.Cu at (65.6, 43.2)
- added C10: 0.1u, Capacitor_SMD:C_0402_1005Metric, F.Cu at (-109.4, 31.7)
- added C10: 0.1u, Capacitor_SMD:C_0402_1005Metric, F.Cu at (61.9, 55.6)
- added C12: 0.1u, Capacitor_SMD:C_0402_1005Metric, F.Cu at (-113.1, 52.0)
- added C12: 0.1u, Capacitor_SMD:C_0402_1005Metric, F.Cu at (65.6, 35.3)
- added C14: 0.1u, Capacitor_SMD:C_0402_1005Metric, F.Cu at (-113.1, 54.1)
- added C14: 0.1u, Capacitor_SMD:C_0402_1005Metric, F.Cu at (65.6, 33.3)
- added C15: 1u, Capacitor_SMD:C_0603_1608Metric, F.Cu at (-116.6, 53.9)
- added C15: 1u, Capacitor_SMD:C_0603_1608Metric, F.Cu at (69.1, 33.5)
- added C19: 0.1u, Capacitor_SMD:C_0402_1005Metric, F.Cu at (-115.1, 59.5)
- added C19: 0.1u, Capacitor_SMD:C_0402_1005Metric, F.Cu at (67.6, 27.9)
- added C2: 0.1u, Capacitor_SMD:C_0402_1005Metric, F.Cu at (-113.1, 50.0)
- added C2: 0.1u, Capacitor_SMD:C_0402_1005Metric, F.Cu at (65.6, 37.4)
- added C20: 0.1u, Capacitor_SMD:C_0402_1005Metric, F.Cu at (-115.1, 57.9)
- added C20: 0.1u, Capacitor_SMD:C_0402_1005Metric, F.Cu at (67.6, 29.5)
- added C22: 10u, Capacitor_SMD:C_0805_2012Metric, F.Cu at (77.6, 45.3)
- added C23: 0.1u, Capacitor_SMD:C_0402_1005Metric, F.Cu at (27.4, 44.4)
- added C24: 18p, Capacitor_SMD:C_0603_1608Metric, F.Cu at (-116.6, 44.8)
- added C24: 18p, Capacitor_SMD:C_0603_1608Metric, F.Cu at (69.1, 42.6)
- added C25: 18p, Capacitor_SMD:C_0603_1608Metric, F.Cu at (-116.6, 50.6)
- added C25: 18p, Capacitor_SMD:C_0603_1608Metric, F.Cu at (69.1, 36.8)
- added C26: 12.5p, Capacitor_SMD:C_0603_1608Metric, F.Cu at (-115.1, 37.3)
- added C27: 12.5p, Capacitor_SMD:C_0603_1608Metric, F.Cu at (-115.1, 42.9)
- added C27: 12.5p, Capacitor_SMD:C_0603_1608Metric, F.Cu at (67.6, 44.5)
- added C3: 0.1u, Capacitor_SMD:C_0402_1005Metric, F.Cu at (-108.0, 58.1)
- added C3: 0.1u, Capacitor_SMD:C_0402_1005Metric, F.Cu at (60.5, 29.2)
- added C4: 0.1u, Capacitor_SMD:C_0402_1005Metric, F.Cu at (-101.4, 58.1)
- added C4: 0.1u, Capacitor_SMD:C_0402_1005Metric, F.Cu at (53.9, 29.2)
- added C5: 0.1u, Capacitor_SMD:C_0402_1005Metric, F.Cu at (-96.6, 58.1)
- added C5: 0.1u, Capacitor_SMD:C_0402_1005Metric, F.Cu at (49.1, 29.2)
- added C6: 0.1u, Capacitor_SMD:C_0402_1005Metric, F.Cu at (-86.9, 48.8)
- added C6: 0.1u, Capacitor_SMD:C_0402_1005Metric, F.Cu at (39.4, 38.6)
- added C7: 0.1u, Capacitor_SMD:C_0402_1005Metric, F.Cu at (-86.9, 36.6)
- added C7: 0.1u, Capacitor_SMD:C_0402_1005Metric, F.Cu at (39.4, 50.8)
- added C8: 0.1u, Capacitor_SMD:C_0402_1005Metric, F.Cu at (-96.8, 32.2)
- added C8: 0.1u, Capacitor_SMD:C_0402_1005Metric, F.Cu at (49.3, 55.1)
- added C9: 0.1u, Capacitor_SMD:C_0402_1005Metric, F.Cu at (-101.9, 32.2)
- added C9: 0.1u, Capacitor_SMD:C_0402_1005Metric, F.Cu at (54.4, 55.1)
- added J7: PWR_CON, Connector_PinSocket_1.27mm:PinSocket_2x05_P1.27mm_Vertical_SMD, F.Cu at (233.7, 53.3)
- added J7: PWR_CON, Connector_PinSocket_1.27mm:PinSocket_2x05_P1.27mm_Vertical_SMD, F.Cu at (220.2, 53.3)
- added J7: PWR_CON, Connector_PinSocket_1.27mm:PinSocket_2x05_P1.27mm_Vertical_SMD, F.Cu at (188.5, 51.1)
- added JP1: SolderBridge, Jumper:SolderJumper-2_P1.3mm_Open_TrianglePad1.0x1.5mm, F.Cu at (-114.1, 35.3)
- added JP2: SolderBridge, Jumper:SolderJumper-2_P1.3mm_Open_TrianglePad1.0x1.5mm, F.Cu at (-85.7, 42.9)
- added R1: 0, Resistor_SMD:R_0603_1608Metric, F.Cu at (-113.2, 58.7)
- added R2: 0, Resistor_SMD:R_0603_1608Metric, F.Cu at (-114.3, 53.2)
- added R6: 10k, Resistor_SMD:R_0603_1608Metric, F.Cu at (-106.5, 31.2)
- added R7: 10k, Resistor_SMD:R_0603_1608Metric, F.Cu at (-104.9, 31.2)
- added R7: 10k, Resistor_SMD:R_0603_1608Metric, F.Cu at (57.4, 56.2)
- added R8: 10k, Resistor_SMD:R_0603_1608Metric, F.Cu at (-108.0, 31.2)
- added U2: STM32H743ZITx, Package_QFP:LQFP-144_20x20mm_P0.5mm, F.Cu at (-99.9, 45.2)
- added Y1: 8M RH100-8.000-20-3050-EXT-TR, Crystal:Crystal_SMD_3225-4Pin_3.2x2.5mm, F.Cu at (-116.5, 47.7)
- added Y1: 8M RH100-8.000-20-3050-EXT-TR, Crystal:Crystal_SMD_3225-4Pin_3.2x2.5mm, F.Cu at (69.0, 39.7)
- added Y2: 32k FC-135 32.7680KA-A0, Crystal:Crystal_SMD_3215-2Pin_3.2x1.5mm, F.Cu at (-115.1, 40.1)
- C11: value 0.1u -> 4.7u
- C13, C16: value 0.1u -> 1u
- C17: value 1u -> 2.2u
- C18: value 0.1u -> 2.2u
- D4: value D_ESD -> ESDALC6V1-1U2; footprint Diode_SMD:D_MELF -> Diode_SMD:D_0201_0603Metric
- D5, D6, D7: value SBD -> SBD RB520S; footprint Diode_SMD:D_MELF -> Diode_SMD:D_0603_1608Metric
- SW1: value RST_SW -> SW_RESET
- moved C13 295.7 mm to (-116.6, 52.4), turned to 180 degrees
- moved C16 284.7 mm to (-112.8, 38.1), turned to 90 degrees
- moved C17 239.3 mm to (-85.9, 38.3)
- moved C11 213.9 mm to (-85.1, 36.0), turned to 270 degrees
- moved C18 209.8 mm to (-91.6, 59.2), turned to 270 degrees
- moved J1 132.2 mm to (32.5, 58.2), turned to 0 degrees
- moved C18 129.0 mm to (44.1, 28.2), turned to 90 degrees
- moved R8 114.7 mm to (60.5, 56.2), turned to 270 degrees
- moved R6 111.9 mm to (59.0, 56.2), turned to 90 degrees
- moved C16 106.6 mm to (65.3, 49.2), turned to 270 degrees
- moved C13 102.0 mm to (69.1, 35.0)
- moved U2 99.2 mm to (52.4, 42.2), turned to 180 degrees
- moved JP2 97.3 mm to (38.3, 44.4)
- moved D13 96.0 mm to (40.0, 60.2)
- moved C11 84.8 mm to (37.6, 51.4), turned to 90 degrees
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- renumbered C1 to C11, C14 to C13, C19 to C16, C22 to C17, C23 to C18, R7 to R8
Connections:
- C11 pad 1: /3V3_VDD -> (no net)
- C11 pad 2: GND -> (no net)
- C13 pad 1: /3V3_VDD -> (no net)
- C13 pad 2: GND -> (no net)
- C16 pad 1: /3V3_VDD -> (no net)
- C16 pad 2: GND -> (no net)
- C17 pad 1: /VDDA -> (no net)
- C17 pad 2: GND -> (no net)
- C18 pad 1: /3V3_VDD -> (no net)
- C18 pad 2: GND -> (no net)
- C21 pad 1: /NJTRST -> /5V_IN
Routing:
- net GND: track 0.00 -> 178.1 mm, vias 0 -> 4
- net (no net): track 0.00 -> 174.8 mm
- net /3V3_VDD: track 0.00 -> 103.9 mm
- net /NJTRST: track 0.00 -> 77.6 mm, vias 0 -> 2
- net /SPI5_NSS: track 0.00 -> 58.1 mm, vias 0 -> 2
- net /Culc_PIN: track 0.00 -> 51.5 mm, vias 0 -> 6
- net /OC_MODE: track 0.00 -> 50.4 mm, vias 0 -> 2
- net /PWM_MODE: track 0.00 -> 49.9 mm, vias 0 -> 2
- net /SPI5_SCK: track 0.00 -> 48.2 mm, vias 0 -> 2
- net /ABZ_ENC_A: track 0.00 -> 47.8 mm, vias 0 -> 2
- net /ABZ_ENC_GPIO: track 0.00 -> 43.1 mm, vias 0 -> 2
- net /ADC_W: track 0.00 -> 43.0 mm, vias 0 -> 2
- net /ABZ_ENC_B: track 0.00 -> 42.6 mm, vias 0 -> 2
- net /Gate_Enable: track 0.00 -> 42.6 mm, vias 0 -> 2
- net /UART_TX: track 0.00 -> 41.8 mm, vias 0 -> 2
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Other:
- board outline added: 234.9 x 114.3 mm
- net class FusionPCB added: clearance 0.18, trace_width 0.18, via_dia 0.8, via_drill 0.4
- rule trace_min: 0.2 -> 0.1524
- rule via_min_size: 0.4 -> 0.7
